File: melvins board.brd (EAGLE design)
At the start: 53.3 x 35.6 mm, 9 parts, among them J2 6_PIN_SERIAL_CABLEPTH, U1 328P

Commit message: Added the right ones
Parts:
- moved FRAME1 4.02 mm to (-78.7, 29.2)
- moved J1 3.81 mm to (108.0, 25.4)
- moved Y2 2.54 mm to (95.2, 25.4)
- moved C1 1.27 mm to (88.9, 34.3)
Routing:
- net GND: track 126.0 -> 98.7 mm
- net 5V: track 146.5 -> 138.9 mm
- net N$2: track 21.5 -> 20.4 mm
- net N$3: track 18.8 -> 17.9 mm
Other:
- board size 53.3 x 35.6 mm -> 52.1 x 33 mm
